File: mosfet.sch (KiCad schematic (older format))
At the start: 5 parts, among them Q1 Q_NMOS_SGD, U5 MIC5060

Commit message: Assign footprints
Parts:
- C23: footprint (none) -> Capacitor_SMD:C_0603_1608Metric_Pad1.05x0.95mm_HandSolder
- C24: footprint (none) -> Capacitor_SMD:C_0805_2012Metric_Pad1.15x1.40mm_HandSolder
- Q1: value Q_NMOS_SGD -> IRF8734; footprint (none) -> extraFootprints:SOIC-8-MOSFET
- R14: footprint (none) -> Resistor_SMD:R_0603_1608Metric_Pad1.05x0.95mm_HandSolder
- U5: footprint (none) -> Package_DFN_QFN:MLF-8-1EP_3x3mm_P0.65mm_EP1.55x2.3mm
Changed lines of the file:
@@
 F 0 "U5" H 4900 3715 50  0000 C CNN
 F 1 "MIC5060" H 4900 3624 50  0000 C CNN
-F 2 "" H 5200 3100 50  0001 C CNN
+F 2 "Package_DFN_QFN:MLF-8-1EP_3x3mm_P0.65mm_EP1.55x2.3mm" H 5200 3100 50  0001 C CNN
 F 3 "http://ww1.microchip.com/downloads/en/DeviceDoc/mic5060.pdf" H 5200 3100 50  0001 C CNN
 	1    4900 3350
@@
 AR Path="/5F22CDBC/5F278D24" Ref="Q3"  Part="1"
 F 0 "Q1" H 6154 3246 50  0000 L CNN
-F 1 "Q_NMOS_SGD" H 6154 3155 50  0000 L CNN
-F 2 "" H 6150 3300 50  0001 C CNN
-F 3 "~" H 5950 3200 50  0001 C CNN
+F 1 "IRF8734" H 6154 3155 50  0000 L CNN
+F 2 "extraFootprints:SOIC-8-MOSFET" H 6150 3300 50  0001 C CNN
+F 3 "https://www.infineon.com/dgdl/irf8734pbf.pdf?fileId=5546d462533600a40153560d97fd1d7d" H 5950 3200 50  0001 C CNN
 	1    5950 3200
 	1    0    0    -1
@@
 F 0 "R14" V 5343 3200 50  0000 C CNN
 F 1 "10R" V 5434 3200 50  0000 C CNN
-F 2 "" V 5480 3200 50  0001 C CNN
+F 2 "Resistor_SMD:R_0603_1608Metric_Pad1.05x0.95mm_HandSolder" V 5480 3200 50  0001 C CNN
 F 3 "~" H 5550 3200 50  0001 C CNN
 	1    5550 3200
@@
 F 0 "C24" H 4050 3450 50  0000 L CNN
 F 1 "10u" H 4050 3250 50  0000 L CNN
-F 2 "" H 4038 3200 50  0001 C CNN
+F 2 "Capacitor_SMD:C_0805_2012Metric_Pad1.15x1.40mm_HandSolder" H 4038 3200 50  0001 C CNN
 F 3 "~" H 4000 3350 50  0001 C CNN
 	1    4000 3350
@@
 F 0 "C23" H 3800 3450 50  0000 L CNN
 F 1 "100n" H 3800 3250 50  0000 L CNN
-F 2 "" H 3788 3200 50  0001 C CNN
+F 2 "Capacitor_SMD:C_0603_1608Metric_Pad1.05x0.95mm_HandSolder" H 3788 3200 50  0001 C CNN
 F 3 "~" H 3750 3350 50  0001 C CNN
 	1    3750 3350

Commit message: Finish PCB
Parts:
- removed R14: 10R, Resistor_SMD:R_0603_1608Metric_Pad1.05x0.95mm_HandSolder, symbol Device:R
Connections:
- net +24V is gone; now on net Voltage_In: C23.1, C24.1, U5.1 (VDD)
- net at U5.5 (Gate): now also Q1.2 (G)
Changed lines of the file:
@@
 $EndComp
-$Comp
-L Device:R R14
-U 1 1 5F27B9C2
-P 5550 3200
-AR Path="/5F277E83/5F27B9C2" Ref="R14"  Part="1"
-AR Path="/5F28697D/5F27B9C2" Ref="R?"  Part="1"
-AR Path="/5F292969/5F27B9C2" Ref="R?"  Part="1"
-AR Path="/5F220C8C/5F27B9C2" Ref="R15"  Part="1"
-AR Path="/5F22CDBC/5F27B9C2" Ref="R16"  Part="1"
-F 0 "R14" V 5343 3200 50  0000 C CNN
-F 1 "10R" V 5434 3200 50  0000 C CNN
-F 2 "Resistor_SMD:R_0603_1608Metric_Pad1.05x0.95mm_HandSolder" V 5480 3200 50  0001 C CNN
-F 3 "~" H 5550 3200 50  0001 C CNN
-	1    5550 3200
-	0    1    1    0
-$EndComp
-Wire Wire Line
-	5750 3200 5700 3200
 $Comp
 L power:GND #PWR033
@@
 AR Path="/5F220C8C/5F27CECC" Ref="#PWR035"  Part="1"
 AR Path="/5F22CDBC/5F27CECC" Ref="#PWR037"  Part="1"
-F 0 "#PWR033" H 4450 3350 50  0001 C CNN
+F 0 "#PWR037" H 4450 3350 50  0001 C CNN
 F 1 "GND" H 4455 3427 50  0000 C CNN
 F 2 "" H 4450 3600 50  0001 C CNN
@@
 Wire Wire Line
 	6050 2950 6050 3000
-$Comp
-L power:+24V #PWR032
-U 1 1 5F27D3C9
-P 4450 3100
-AR Path="/5F277E83/5F27D3C9" Ref="#PWR032"  Part="1"
-AR Path="/5F28697D/5F27D3C9" Ref="#PWR?"  Part="1"
-AR Path="/5F292969/5F27D3C9" Ref="#PWR?"  Part="1"
-AR Path="/5F220C8C/5F27D3C9" Ref="#PWR034"  Part="1"
-AR Path="/5F22CDBC/5F27D3C9" Ref="#PWR036"  Part="1"
-F 0 "#PWR032" H 4450 2950 50  0001 C CNN
-F 1 "+24V" H 4465 3273 50  0000 C CNN
-F 2 "" H 4450 3100 50  0001 C CNN
-F 3 "" H 4450 3100 50  0001 C CNN
-	1    4450 3100
-	1    0    0    -1
-$EndComp
 Wire Wire Line
 	4500 3250 4450 3250
@@
 Connection ~ 4450 3150
 Wire Wire Line
-	4450 3150 4450 3100
-Wire Wire Line
 	4000 3500 4000 3550
 Wire Wire Line
@@
 Wire Wire Line
 	4450 3550 4450 3450
-Text HLabel 6050 3550 3    50   Input ~ 0
+Text HLabel 6050 3550 3    50   Output ~ 0
 LOAD
 Text HLabel 4450 3350 0    50   Input ~ 0
@@
 Wire Wire Line
 	5350 3250 5350 3200
-Wire Wire Line
-	5350 3200 5400 3200
 Connection ~ 6050 3450
 Wire Wire Line
@@
 Text HLabel 6050 2950 1    50   Input ~ 0
 Voltage_In
+Wire Wire Line
+	5350 3200 5750 3200
+Text HLabel 4450 3050 1    50   Input ~ 0
+Voltage_In
+Wire Wire Line
+	4450 3050 4450 3150
 $EndSCHEMATC
